File: ODrive.kicad_pcb (KiCad board)
At the start: 4 copper layers, 53 x 70 mm, 162 parts, among them J1 Conn_01x02_Pin, J10 Conn_01x02_Pin, J11 Conn_01x05_Pin, J12 Conn_01x04_Pin, J13 Conn_01x06_Pin, J2 Conn_01x02_Pin, J3 Conn_01x02_Pin, J4 USB_C_Receptacle_USB2.0_16P, J5 Conn_01x02_Pin, J6 Conn_01x04_Pin, J7 Conn_01x03_Pin, J8 Conn_01x05_Pin, J9 Conn_01x03_Pin, Q1 NTMFS5C628NLT1G, Q10 NTMFS5C628NLT1G, Q11 NTMFS5C628NLT1G, Q12 NTMFS5C628NLT1G, Q13 NTMFS5C628NLT1G, Q14 NTMFS5C628NLT1G, Q2 NTMFS5C628NLT1G, Q3 NTMFS5C628NLT1G, Q4 NTMFS5C628NLT1G, Q5 NTMFS5C628NLT1G, Q6 NTMFS5C628NLT1G, Q7 NTMFS5C628NLT1G, Q8 NTMFS5C628NLT1G, Q9 NTMFS5C628NLT1G, SW1 SW_DIP_x01, SW2 SW_DIP_x01, U1 MIC5524-3.3YMT-T5, U2 LM5109BMA, U3 STM32F405RGTx, U4 DRV8301DCAR, U5 DRV8301DCAR, U6 SN65HVD1050D, Y2 Crystal_GND24_Small

Commit message: 0.4/0.3
Parts:
- moved R15 0.08 mm to (14.4, 29.5)
Routing:
- net /M1_AL: track 29.0 -> 58.2 mm
- net /M0_CH: track 23.7 -> 28.5 mm
- net GND: track 221.2 -> 225.6 mm, vias 197 -> 196
- net /M0_ENC_Z: track 37.3 -> 40.8 mm
- net /M0_BL: track 28.1 -> 31.2 mm
- net /SPI_MISO: track 44.2 -> 47.2 mm
- net /nFAULT: track 42.9 -> 45.8 mm
- net /SPI_MOSI: track 44.2 -> 47.1 mm
- net /M1_CL: track 28.3 -> 30.9 mm
- net /M0_SO1: track 34.7 -> 37.1 mm
- net /M1/SL_C: track 29.9 -> 32.0 mm
- net /M1_SO2: track 18.9 -> 21.0 mm
- net /M1_TEMP: track 39.4 -> 41.3 mm
- net +5V: track 56.4 -> 54.5 mm
- net /SPI_SCK : track 44.6 -> 46.5 mm
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Other:
- board text added: "+"
- board text added: "-"
- board text added: "A"
- board text added: "B"
- board text added: "BRAKE"
- board text added: "C"
- board text added: "CAN END"
- board text added: "D"
- board text added: "ENC0"
- board text added: "ENC1"
- board text added: "G"
- board text added: "G EN DIR STEP"
- board text added: "H"
- board text added: "JLCJLCJLC"
- board text added: "L"
- board text added: "M0"
- board text added: "M1"
- board text added: "R"
- board text added: "T"
