File: ODrive.kicad_sch (KiCad schematic)
At the start: 76 parts, among them J1 Conn_01x02_Pin, J10 Conn_01x02_Pin, J11 Conn_01x05_Pin, J12 Conn_01x04_Pin, J13 Conn_01x06_Pin, J2 Conn_01x02_Pin, J3 Conn_01x02_Pin, J4 USB_C_Receptacle_USB2.0_16P, J5 Conn_01x02_Pin, J6 Conn_01x04_Pin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

Commit message: x
Parts:
- R11: value 10k -> 1.3k
- R12: value 10k -> 18k
- R13: value 10k -> 8.2k
- R14: value 10k -> 43k
Other:
- note added: "V_ref = 0.8"
Changed lines of the file:
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@@
     (stroke (width 0) (type default))
   )
+  (text "V_ref = 0.8" (at 226.06 87.63 0)
+    (effects (font (size 1.27 1.27)) (justify left bottom))
+  )
+  (text "V_ref = 0.8" (at 226.06 138.43 0)
+    (effects (font (size 1.27 1.27)) (justify left bottom))
+  )
   (label "M0_C" (at 228.6 67.31 0) (fields_autoplaced)
     (effects (font (size 1.27 1.27)) (justify left bottom))
@@
       (effects (font (size 1.27 1.27)) (justify right))
     )
-    (property "Value" "10k" (at 243.84 97.79 0)
+    (property "Value" "43k" (at 243.84 97.79 0)
       (effects (font (size 1.27 1.27)) (justify right))
     )
@@
       (effects (font (size 1.27 1.27)) (justify right))
     )
-    (property "Value" "10k" (at 243.84 87.63 0)
+    (property "Value" "8.2k" (at 243.84 87.63 0)
       (effects (font (size 1.27 1.27)) (justify right))
     )
@@
       (effects (font (size 1.27 1.27)) (justify right))
     )
-    (property "Value" "10k" (at 242.57 138.43 0)
+    (property "Value" "1.3k" (at 242.57 138.43 0)
       (effects (font (size 1.27 1.27)) (justify right))
     )
@@
       (effects (font (size 1.27 1.27)) (justify right))
     )
-    (property "Value" "10k" (at 242.57 148.59 0)
+    (property "Value" "18k" (at 242.57 148.59 0)
       (effects (font (size 1.27 1.27)) (justify right))
     )
